File: pcb/pcb.kicad_pcb (KiCad board)
At the start: 2 copper layers, 422.8 x 128.1 mm, 299 parts, among them SW1 RotaryEncoder_Switch

Commit message: Updated PCB slightly
Other:
- board text added: "Something fucked up, huh?"
- board text added: "You have voided your warranty by seeing this."
Changed lines of the file:
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@@
 		(layer "Edge.Cuts")
+	)
+	(gr_text "You have voided your warranty by seeing this."
+		(at 379 149.5 0)
+		(layer "Edge.Cuts")
+		(effects
+			(font
+				(size 1.5 1.5)
+				(thickness 0.25)
+				(bold yes)
+			)
+			(justify left bottom)
+		)
+	)
+	(gr_text "Something fucked up, huh?"
+		(at 490.2 105.15 90)
+		(layer "Edge.Cuts")
+		(effects
+			(font
+				(size 1 1)
+				(thickness 0.15)
+			)
+			(justify left bottom)
+		)
 	)
 	(segment
